File: PCB/ServoTester1822.sch (KiCad schematic (older format))
At the start: 26 parts, among them IC1 PIC12(L)F1822-I/P, P1 CONN_01X02, P2 CONN_01X03, P3 CONN_01X03, SW1 SW_PUSH, SW2 SW_PUSH, SW3 SW_PUSH, SW4 SW_PUSH, U1 7805

Commit message: Started PCB
Parts:
- C1: footprint (none) -> Capacitors_Elko_ThroughHole:Elko_vert_11x5mm_RM2.5
- C2, C3, C4: footprint (none) -> Capacitors_SMD:C_0805_HandSoldering
- D1: footprint (none) -> Diodes_SMD:Diode-SMA_Handsoldering
- D2, D3, D4: footprint (none) -> LEDs:LED-1206
- IC1: footprint (none) -> Housings_DIP:DIP-8_W7.62mm
- P1: footprint (none) -> Connect:bornier2
- P2: footprint (none) -> Connect:bornier3
- P3: footprint (none) -> Pin_Headers:Pin_Header_Straight_1x03
- R1, R2, R3, R4, R5, R6, R7, R8: footprint (none) -> Resistors_SMD:R_0805_HandSoldering
- SW1, SW2, SW3, SW4: footprint (none) -> Buttons_Switches_SMD:SW_SPST_PTS645
- U1: footprint (none) -> TO_SOT_Packages_THT:TO-220_Neutral123_Vertical
