File: PCB/ServoTester1822.kicad_pcb (KiCad board)
At the start: 2 copper layers, 25 parts, among them IC1 PIC12(L)F1822-I/P, P1 CONN_01X02, P2 CONN_01X03, P3 CONN_01X03, SW1 SW_PUSH, SW2 SW_PUSH, SW3 SW_PUSH, SW4 SW_PUSH, U1 7805

Commit message: Ordered PCB
Parts:
- added H1: MountingHole_2-7mm, Mounting_Holes:MountingHole_2-7mm, F.Cu at (152.4, 102.2)
- added H2: MountingHole_2-7mm, Mounting_Holes:MountingHole_2-7mm, F.Cu at (106.7, 134.0)
- added RV1: 20K, PTV09A:PTV09A-1, F.Cu at (116.2, 118.2)
- moved C1 45.9 mm to (115.6, 109.2), turned to 270 degrees
- moved C2 45.8 mm to (111.8, 128.9), turned to 90 degrees
- moved P2 42.5 mm to (144.1, 132.7)
- moved R6 40.4 mm to (132.6, 133.3), turned to 180 degrees
- moved C3 39.6 mm to (125.1, 112.4), turned to 180 degrees
- moved SW1 38.4 mm to (125.6, 117.8)
- moved P1 35.9 mm to (108.0, 106.0), turned to 270 degrees
- moved C4 33.7 mm to (132.7, 129.5)
- moved D2 30.9 mm to (141.0, 110.0), turned to 270 degrees
- moved SW3 29.4 mm to (149.4, 117.2)
- moved SW4 28.8 mm to (149.4, 124.8)
- moved D3 26.7 mm to (141.0, 117.6), turned to 270 degrees
- moved R3 26.1 mm to (135.3, 111.1)
- moved P3 25.8 mm to (132.1, 103.5), turned to 90 degrees
- moved U1 22.9 mm to (123.8, 109.2)
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Routing:
- net GND: track 0.00 -> 173.9 mm
- net +5V: track 0.00 -> 108.2 mm, vias 0 -> 2
- net Net-(D2-Pad1): track 0.00 -> 87.7 mm, vias 0 -> 1
- net Net-(D3-Pad1): track 0.00 -> 50.6 mm, vias 0 -> 1
- net Net-(D4-Pad1): track 0.00 -> 46.4 mm
- net Net-(P3-Pad1): track 0.00 -> 31.7 mm, vias 0 -> 1
- net Net-(IC1-Pad4): track 0.00 -> 24.1 mm, vias 0 -> 1
- net Net-(C4-Pad1): track 0.00 -> 22.6 mm
- net Net-(IC1-Pad2): track 0.00 -> 13.1 mm
- net Net-(C1-Pad1): track 0.00 -> 13.0 mm
- net Net-(D1-Pad2): track 0.00 -> 8.23 mm
- net Net-(D4-Pad2): track 0.00 -> 4.41 mm
- net Net-(D3-Pad2): track 0.00 -> 4.41 mm
- net Net-(D2-Pad2): track 0.00 -> 4.41 mm
Other:
- board outline added: 52.1 x 38.1 mm
- net class Default: trace_width 0.25 -> 0.3048; via_dia 0.6 -> 1.016; via_drill 0.4 -> 0.5588
- rule pad_to_mask_clearance: 0.2 -> 0
- board text added: "+6V"
- board text added: "Alpha"
- board text added: "Beta"
- board text added: "C + -"
- board text added: "Center"
- board text added: "GND"
- board text added: "Optional I2C"
- board text added: "Servo"
- board text added: "Servo Tester 1822 DMFE 2015"
